File: Keyboard Memory Emulator/Keyboard Memory Emulator.kicad_pcb (KiCad board)
At the start: 2 copper layers, 40 parts, among them J1 Conn_01x05, J2 Conn_01x01_Male, J3 Conn_01x02, J4 Conn_01x03, J5 Conn_01x02, J6 Conn_01x04, J7 Conn_01x05, J8 Conn_02x05_Odd_Even, SW1 PTS636 SL43 LFS, U1 SN74HC244APWR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

Commit message: Added labels on PCB, and adjusted font sizes to match jlcpcb's requirements.
Other:
- board text added: "100n"
- board text added: "10K"
- board text added: "12.5p"
- board text added: "32.768kHz"
- board text added: "A0"
- board text added: "A1"
- board text added: "A10"
- board text added: "A11"
- board text added: "A12"
- board text added: "A13"
- board text added: "A2"
- board text added: "A3"
- board text added: "A4"
- board text added: "A5"
- board text added: "A6"
- board text added: "A7"
- board text added: "A8"
- board text added: "A9"
- board text added: "CS"
- board text added: "D0"
- board text added: "D1"
- board text added: "D2"
- board text added: "D3"
- board text added: "D4"
- board text added: "D5"
- board text added: "D6"
- board text added: "D7"
- board text added: "NC"
- board text added: "OE"
- board text added: "T"
- board text added: "WE"
- board text removed: "5v"

Commit message: Added a gitignore, hopefully it will work as I hope. I also fixed the traces that were not showing up due to improper nets.
Connections:
- U6 pad 27: Net-(U6-Pad27) -> /GWE
